File: HeadlightDimmerPCB.kicad_sch (KiCad schematic)
At the start: 12 parts, among them J1 Conn_02x02_Counter_Clockwise, Q1 NMOS, U1 LMC555xTP

Commit message: bah
Parts:
- removed U1: LMC555xTP, Package_BGA:Texas_DSBGA-8_1.43x1.41mm_Layout3x3_P0.5mm, symbol Timer:LMC555xTP
- added U1: LMC555xM, Package_SO:SOIC-8_3.9x4.9mm_P1.27mm, symbol Timer:LMC555xM
- C1, C2: footprint Capacitor_SMD:C_0603_1608Metric -> Capacitor_SMD:C_0805_2012Metric_Pad1.18x1.45mm_HandSolder
- D1, D2: footprint Diode_SMD:D_0603_1608Metric_Pad1.05x0.95mm_HandSolder -> Diode_SMD:D_0805_2012Metric_Pad1.15x1.40mm_HandSolder
- R1, R2, R3: footprint Resistor_SMD:R_0603_1608Metric -> Resistor_SMD:R_0805_2012Metric_Pad1.20x1.40mm_HandSolder
Connections:
- net VBC is gone; now on net VDC: R1.2
- net DIS: now also U1.7 (DIS)
- net GNDPWR: now also U1.1 (GND)
- net VDC: now also U1.4 (R), U1.8 (VCC)
- net at C2.1, RV1.2: now also U1.2 (TR), U1.6 (THR)
- net at C1.1: now also U1.5 (CV)
- net at R2.1: now also U1.3 (Q)

Commit message: more routing and part selection
Parts:
- removed D1, D2: D, Diode_SMD:D_0805_2012Metric_Pad1.15x1.40mm_HandSolder, symbol Device:D
- added D3: BAT54V-7, Package_TO_SOT_SMD:SOT-563, symbol BAT54V-7:BAT54V-7
- C1: P/N (none) -> C0805C103M5RACTU
- C2: P/N (none) -> C3216C0G2J103G160AE
- F1: P/N (none) -> JB12F2001R
- Q1: P/N (none) -> DMG2302UKQ-7
- R1: P/N (none) -> CRCW08051K00FKEAC
- R2: value 100 -> 1K; P/N (none) -> CRCW08051K00FKEAC
- R3: value 10k -> 10K; P/N (none) -> CRCW080510K0FKEAC
- RV1: value 10k -> 10K; P/N (none) -> PS10KH40-103A3030
- U1: P/N (none) -> LMC555xM
Connections:
- net DIS: now also D3.3 (C2), D3.4 (A2)
- net at RV1.1: now also D3.6 (C1)
- net at RV1.3: now also D3.1 (A1)
- no-connect marks 0 -> 2
Other:
- note added: "Pot varies duty cycle D = 1 - RV1/(11k) T = ln2 * (11k) (0.01uF) = 0.00007624618 S = 76.25 uS f = 13.1147541 kHz https://electronics.stackexchange.com/questions/563128/555-timer-duty-cycle-changing-formula"
- moved on the sheet: C1, C2, F1, J1, Q1, R1, R2, R3, RV1, U1

Commit message: final
Parts:
- D3: P/N (none) -> BAT54V
Changed lines of the file:
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@@
+	)
+	(junction
+		(at 85.09 59.69)
+		(diameter 0)
+		(color 0 0 0 0)
 	)
 	(junction
@@
 	)
 	(junction
-		(at 88.9 59.69)
-		(diameter 0)
-		(color 0 0 0 0)
-	)
-	(junction
 		(at 102.87 59.69)
 		(diameter 0)
@@
 	(wire
 		(pts
-			(xy 175.26 72.39) (xy 119.38 72.39)
-		)
-		(stroke
-			(width 0)
-			(type default)
-		)
-	)
-	(wire
-		(pts
-			(xy 167.64 100.33) (xy 175.26 100.33)
+			(xy 176.53 72.39) (xy 119.38 72.39)
+		)
+		(stroke
+			(width 0)
+			(type default)
+		)
+	)
+	(wire
+		(pts
+			(xy 167.64 100.33) (xy 176.53 100.33)
 		)
 		(stroke
@@
 	(wire
 		(pts
-			(xy 88.9 59.69) (xy 102.87 59.69)
-		)
-		(stroke
-			(width 0)
-			(type default)
-		)
-	)
-	(wire
-		(pts
 			(xy 149.86 138.43) (xy 149.86 130.81)
 		)
@@
 	(wire
 		(pts
-			(xy 85.09 59.69) (xy 88.9 59.69)
+			(xy 85.09 59.69) (xy 102.87 59.69)
 		)
 		(stroke
@@
 	(wire
 		(pts
-			(xy 175.26 100.33) (xy 175.26 72.39)
+			(xy 176.53 100.33) (xy 176.53 72.39)
 		)
 		(stroke
@@
 	(wire
 		(pts
-			(xy 88.9 55.88) (xy 88.9 59.69)
+			(xy 85.09 55.88) (xy 85.09 59.69)
 		)
 		(stroke
@@
 	)
 	(label "DIS"
-		(at 88.9 55.88 0)
+		(at 85.09 55.88 0)
 		(effects
 			(font
@@
 				(hide yes)
 			)
+		)
+		(property "P/N" "BAT54V"
+			(at 86.36 71.12 0)
+			(effects
+				(font
+					(size 1.27 1.27)
+				)
+				(hide yes)
+			)
